File: delayed_pulser.sch (EAGLE design)
At the start: 36 parts, among them T1 2N2369, U1 MC100EP196FAG, U2 MC100EPT22DG, U3 MC100EPT22DG, X1 BU-SMA-H, X2 BU-SMA-H, X3 BU-SMA-H, X4 BU-SMA-H

Commit message: added delayed pulse generator, only avalanche transistor for now
Other:
- note added: "Copyright 2015 by Mathias Helsen, MIT license"
Changed lines of the file:
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@@
 <sheet>
 <plain>
+<text x="-30.48" y="55.88" size="1.778" layer="91">Copyright 2015 by Mathias Helsen, MIT license</text>
 </plain>
 <instances>

Commit message: added HV supply
Parts:
- added C13, C14: 0.47, resistor:C-EU050-035X075
- added C15: (no value), resistor:C-EUC1206
- added D1, D2, D3: ES2D, diode:ES2D
- added JP4: (no value), pinhead:PINHD-1X3
- added R11: 1M, resistor:R-EU_M0805
- added R12: (no value), resistor:R-EU_M0805
- added R13: (no value), resistor:R-TRIMMT18
- added R15: 220, resistor:R-EU_M0805
- added U$3: LT1073, LT1073:LT1073
- C11, C12: value (none) -> 8p
- C8: value 4p8 -> 0.47; device resistor:C-EUC0805 -> resistor:C-EU050-035X075
- R14: value Rlim -> 10k
- R3: value 100 -> 200
- R5, R6: value 30 -> 50
Connections:
- new net N$37: C14.2, D1.A, U$3.SW1
- new net N$38: R12.2, R13.A
- new net N$39: R11.1, R13.E
- new net N$40: R13.S, U$3.SENSE
- new net N$41: R15.1, U$3.ILIM
- net +3V3: now also C15.1, JP4.2, R15.2, U$3.VIN
- net GND: now also C13.2, C15.2, C8.2, JP1.2, JP4.1, JP4.3, R12.1, R5.1, R6.2, U$3.GND, U$3.SW2; no longer JP1.1
- net N$11: now also C11.1; no longer C8.2, R5.2
- net N$12: now also C12.1; no longer R6.2
- net N$13: now also C8.1, D1.C, D2.A; no longer JP1.2, R14.2
- net N$24: now also C14.1, D2.C, D3.A; no longer C11.1, R5.1
- net N$25: now also C13.1, D3.C, JP1.1, R11.2, R14.2; no longer C12.1, R6.1
- net N$26: now also R5.2
- net N$27: now also R6.1
- net N$7: no longer C8.1
Other:
- note added: "-> Clipping lines"
- moved on the sheet: C10, C11, C12, C8, JP1, R14, R5, R6, X1

Commit message: added comment
Parts:
- R12: value (none) -> 2k4
- R13: value (none) -> 10k
Other:
- note added: "-> Clipping lines, 100ps long"
- note removed: "-> Clipping lines"
Changed lines of the file:
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@@
 <part name="GND18" library="supply1" deviceset="GND" device=""/>
 <part name="R11" library="resistor" deviceset="R-EU_" device="M0805" value="1M"/>
-<part name="R12" library="resistor" deviceset="R-EU_" device="M0805"/>
-<part name="R13" library="resistor" deviceset="R-TRIMM" device="T18"/>
+<part name="R12" library="resistor" deviceset="R-EU_" device="M0805" value="2k4"/>
+<part name="R13" library="resistor" deviceset="R-TRIMM" device="T18" value="10k"/>
 <part name="GND19" library="supply1" deviceset="GND" device=""/>
 <part name="GND20" library="supply1" deviceset="GND" device=""/>
@@
 <plain>
 <text x="-33.02" y="109.22" size="1.778" layer="97">Copyright 2015 by Mathias Helsen, MIT license</text>
-<text x="124.46" y="60.96" size="1.778" layer="97">-&gt; Clipping lines</text>
+<text x="124.46" y="60.96" size="1.778" layer="97">-&gt; Clipping lines, 100ps long</text>
 </plain>
 <instances>
@@
 <pinref part="U$3" gate="G$1" pin="SENSE"/>
 <wire x1="20.32" y1="68.58" x2="25.4" y2="68.58" width="0.1524" layer="91"/>
-<wire x1="25.4" y1="68.58" x2="25.4" y2="60.96" width="0.1524" layer="91"/>
-<wire x1="25.4" y1="60.96" x2="66.04" y2="60.96" width="0.1524" layer="91"/>
-<wire x1="66.04" y1="60.96" x2="66.04" y2="86.36" width="0.1524" layer="91"/>
+<wire x1="25.4" y1="68.58" x2="25.4" y2="63.5" width="0.1524" layer="91"/>
+<wire x1="25.4" y1="63.5" x2="66.04" y2="63.5" width="0.1524" layer="91"/>
+<wire x1="66.04" y1="63.5" x2="66.04" y2="86.36" width="0.1524" layer="91"/>
 <pinref part="R13" gate="G$1" pin="S"/>
 <wire x1="66.04" y1="86.36" x2="68.58" y2="86.36" width="0.1524" layer="91"/>

Commit message: bla
Parts:
- C13, C14, C8: value 0.47 -> (none); device resistor:C-EU050-035X075 -> resistor:C-EUC0805K
Connections:
- net GND: now also C14.2; no longer C8.2
- net N$13: now also C13.1; no longer C8.1
- net N$24: now also C8.1; no longer C14.1
- net N$25: now also C14.1; no longer C13.1
- net N$37: now also C8.2; no longer C14.2
Other:
- moved on the sheet: C13, C14, C8
Changed lines of the file:
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@@
 <part name="D2" library="diode" deviceset="ES2D" device=""/>
 <part name="D3" library="diode" deviceset="ES2D" device=""/>
-<part name="C8" library="resistor" deviceset="C-EU" device="050-035X075" value="0.47"/>
-<part name="C13" library="resistor" deviceset="C-EU" device="050-035X075" value="0.47"/>
-<part name="C14" library="resistor" deviceset="C-EU" device="050-035X075" value="0.47"/>
 <part name="GND14" library="supply1" deviceset="GND" device=""/>
 <part name="GND18" library="supply1" deviceset="GND" device=""/>
@@
 <part name="JP1" library="pinhead" deviceset="PINHD-1X2" device=""/>
 <part name="GND22" library="supply1" deviceset="GND" device=""/>
+<part name="C8" library="resistor" deviceset="C-EU" device="C0805K"/>
+<part name="C13" library="resistor" deviceset="C-EU" device="C0805K"/>
+<part name="C14" library="resistor" deviceset="C-EU" device="C0805K"/>
 </parts>
 <sheets>
@@
 <instance part="D2" gate="G$1" x="40.64" y="96.52" rot="R90"/>
 <instance part="D3" gate="G$1" x="48.26" y="104.14"/>
-<instance part="C8" gate="G$1" x="40.64" y="81.28"/>
-<instance part="C13" gate="G$1" x="58.42" y="88.9"/>
-<instance part="C14" gate="G$1" x="25.4" y="99.06"/>
 <instance part="GND14" gate="1" x="40.64" y="68.58"/>
 <instance part="GND18" gate="1" x="58.42" y="68.58"/>
@@
 <instance part="JP1" gate="G$1" x="96.52" y="101.6"/>
 <instance part="GND22" gate="1" x="91.44" y="101.6" rot="R270"/>
+<instance part="C8" gate="G$1" x="25.4" y="99.06"/>
+<instance part="C13" gate="G$1" x="40.64" y="81.28"/>
+<instance part="C14" gate="G$1" x="58.42" y="88.9"/>
 </instances>
 <busses>
@@
 </segment>
 <segment>
-<pinref part="C8" gate="G$1" pin="2"/>
 <pinref part="GND14" gate="1" pin="GND"/>
 <wire x1="40.64" y1="71.12" x2="40.64" y2="76.2" width="0.1524" layer="91"/>
-</segment>
-<segment>
 <pinref part="C13" gate="G$1" pin="2"/>
+</segment>
+<segment>
 <pinref part="GND18" gate="1" pin="GND"/>
 <wire x1="58.42" y1="71.12" x2="58.42" y2="83.82" width="0.1524" layer="91"/>
+<pinref part="C14" gate="G$1" pin="2"/>
 </segment>
 <segment>
@@
 <segment>
 <pinref part="D1" gate="G$1" pin="C"/>
-<pinref part="C8" gate="G$1" pin="1"/>
 <wire x1="35.56" y1="88.9" x2="40.64" y2="88.9" width="0.1524" layer="91"/>
 <wire x1="40.64" y1="88.9" x2="40.64" y2="83.82" width="0.1524" layer="91"/>
@@
 <wire x1="40.64" y1="93.98" x2="40.64" y2="88.9" width="0.1524" layer="91"/>
 <junction x="40.64" y="88.9"/>
+<pinref part="C13" gate="G$1" pin="1"/>
 </segment>
 </net>
@@
 <segment>
 <pinref part="D3" gate="G$1" pin="A"/>
-<pinref part="C14" gate="G$1" pin="1"/>
 <wire x1="45.72" y1="104.14" x2="40.64" y2="104.14" width="0.1524" layer="91"/>
 <wire x1="40.64" y1="104.14" x2="25.4" y2="104.14" width="0.1524" layer="91"/>
@@
 <wire x1="40.64" y1="99.06" x2="40.64" y2="104.14" width="0.1524" layer="91"/>
 <junction x="40.64" y="104.14"/>
+<pinref part="C8" gate="G$1" pin="1"/>
 </segment>
 </net>
@@
 <segment>
 <pinref part="D3" gate="G$1" pin="C"/>
-<pinref part="C13" gate="G$1" pin="1"/>
 <wire x1="50.8" y1="104.14" x2="58.42" y2="104.14" width="0.1524" layer="91"/>
 <wire x1="58.42" y1="104.14" x2="58.42" y2="91.44" width="0.1524" layer="91"/>
@@
 <wire x1="93.98" y1="104.14" x2="86.36" y2="104.14" width="0.1524" layer="91"/>
 <junction x="86.36" y="104.14"/>
+<pinref part="C14" gate="G$1" pin="1"/>
 </segment>
 </net>
@@
 <segment>
 <pinref part="D1" gate="G$1" pin="A"/>
-<pinref part="C14" gate="G$1" pin="2"/>
 <wire x1="30.48" y1="88.9" x2="25.4" y2="88.9" width="0.1524" layer="91"/>
 <wire x1="25.4" y1="88.9" x2="25.4" y2="93.98" width="0.1524" layer="91"/>
@@
 <wire x1="25.4" y1="73.66" x2="25.4" y2="88.9" width="0.1524" layer="91"/>
 <junction x="25.4" y="88.9"/>
-</segment>
-</net>
+<pinref part="C8" gate="G$1" pin="2"/>
+</segment>
+</net>

Commit message: finished artwork
Parts:
- removed C14: (no value), resistor:C-EUC0805K
- removed C15: (no value), resistor:C-EUC1206
- removed D1, D2, D3: ES2D, diode:ES2D
- removed R11: 1M, resistor:R-EU_M0805
- removed R12: 2k4, resistor:R-EU_M0805
- removed R13: 10k, resistor:R-TRIMMT18
- removed R15: 220, resistor:R-EU_M0805
- removed U$2: JA4220, \cct:JA4220
- removed U$3: LT1073, LT1073:LT1073
- removed U3: MC100EPT22DG, MC100EPT22:MC100EPT22DG
- added C16, C17: 100p, resistor:C-EUC0603
- added C18, C19: (no value), resistor:C-EUC0805
- added R16: 50, resistor:R-EU_R0805
- C11, C12: value 8p -> 8p2; device resistor:C-EUC0805 -> resistor:C-EUC0603
- C13, C8: device resistor:C-EUC0805K -> resistor:C-EUC0805
- JP3: device pinhead:PINHD-1X4 -> pinhead:PINHD-1X1
- R5, R6: device resistor:R-EU_R0805 -> resistor:R-EU_R0603
Connections:
- removed net N$13: C13.1, D1.C, D2.A
- removed net N$23: U1.SETMIN, U2.Q0
- removed net N$24: C8.1, D2.C, D3.A
- removed net N$25: C14.1, D3.C, JP1.1, R11.2, R14.2
- removed net N$28: U1.SETMAX, U3.Q1
- removed net N$29: U1.~EN, U3.Q0
- removed net N$33: JP3.2, U2.D0
- removed net N$35: JP3.4, U3.D0
- removed net N$36: JP3.3, U3.D1
- removed net N$37: C8.2, D1.A, U$3.SW1
- removed net N$38: R12.2, R13.A
- removed net N$39: R11.1, R13.E
- removed net N$40: R13.S, U$3.SENSE
- removed net N$41: R15.1, U$3.ILIM
- new net VBB: C13.1, C18.1, C19.1, R10.1, R16.1, R7.1, U1.VBB
- net +3V3: now also C8.1; no longer C15.1, R15.2, U$3.VIN, U3.VCC
- net GND: now also C16.2, C17.2, C18.2, C19.2, C8.2, U$1.P$4, U2.D0; no longer C14.2, C15.2, R12.1, U$1.P$1, U$2.P$1, U$2.P$2, U$3.GND, U$3.SW2, U3.GND
- net N$22: now also JP1.1, R14.2; no longer R10.1, R7.1, U1.VBB
- net N$26: now also C16.1; no longer U$2.P$3
- net N$27: now also C17.1; no longer U$2.P$4
- net N$32: now also R16.2
- net N$4: now also U$1.P$2; no longer U$1.P$3
- net N$5: now also U$1.P$3; no longer U$1.P$4
- net N$6: now also U$1.P$1; no longer U$1.P$2
Other:
- moved on the sheet: C10, C11, C12, C13, C2, C4, C8, JP1, R14, R3, R5, R6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
