File: delayed_pulser.brd (EAGLE design)
At the start: 71.1 x 60 mm, 41 parts, among them T1 2N2369, U1 MC100EP196FAG, U2 MC100EPT22DG, X1 BU-SMA-H, X2 BU-SMA-H, X3 BU-SMA-H, X4 BU-SMA-H

Commit message: added prescaled trigger, Work In Progress
Connections:
- net GND: no longer U1.7
Changed lines of the file:
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@@
 <contactref element="R4" pad="1"/>
 <contactref element="JP2" pad="12"/>
-<contactref element="U1" pad="7"/>
 <contactref element="U1" pad="24"/>
 <contactref element="U1" pad="9"/>
