File: prescaled_trigger.sch (EAGLE design)
At the start: 41 parts, among them T1 2N2369, U1 MC100EP196FAG, U2 MC100EPT22DG, X1 BU-SMA-H, X2 BU-SMA-H, X3 BU-SMA-H, X4 BU-SMA-H

Commit message: added prescaled trigger, Work In Progress
Parts:
- removed C10, C13, C18, C19, C8: (no value), resistor:C-EUC0805
- removed C11, C12: 8p2, resistor:C-EUC0603
- removed C16, C17: 100p, resistor:C-EUC0603
- removed C9: (no value), resistor:C-EUC1206
- removed JP1: (no value), pinhead:PINHD-1X2
- removed JP2: (no value), pinhead:PINHD-1X12
- removed JP3: (no value), pinhead:PINHD-1X1
- removed JP4: (no value), pinhead:PINHD-1X3
- removed R14: 10k, resistor:R-EU_R0805
- removed R16: 50, resistor:R-EU_R0805
- removed T1: 2N2369, transistor-neu-to92:2N2369
- removed U1: MC100EP196FAG, MC100EP196:MC100EP196FAG
- removed U2: MC100EPT22DG, MC100EPT22:MC100EPT22DG
- removed X2, X3, X4: BU-SMA-H, con-coax:BU-SMA-H
- added U$2: MC100EP016, MC100EP016:MC100EP016
- R1, R2: value 150 -> 1k; device resistor:R-EU_R0805 -> resistor:R-EU_M0805
- R10, R7: value 50 -> 1k; device resistor:R-EU_R0805 -> resistor:R-EU_M0805
- R3: value 200 -> 50; device resistor:R-EU_R0805 -> resistor:R-EU_M0805
- R4: value 1k -> (none); device resistor:R-EU_R0805 -> resistor:R-TRIMMT18
- R5, R6: value 50 -> (none); device resistor:R-EU_R0603 -> resistor:R-EU_M0805
- R8, R9: value 3k3 -> 1k; device resistor:R-EU_R0805 -> resistor:R-EU_M0805
- U$1: value JA4220 -> MAX9601; device \cct:JA4220 -> MAX9601:MAX9601
Connections:
- removed net N$14: JP2.4, U1.D3
- removed net N$15: JP2.5, U1.D4
- removed net N$16: JP2.6, U1.D5
- removed net N$17: JP2.7, U1.D6
- removed net N$18: JP2.8, U1.D7
- removed net N$19: C10.1, R14.1, R9.2
- removed net N$20: JP2.9, U1.D8
- removed net N$21: JP2.10, U1.D9
- removed net N$22: JP1.1, R14.2
- removed net N$26: C11.2, C16.1, R5.2
- removed net N$27: C12.2, C17.1, R6.1
- removed net N$30: R10.2, U1.~IN, X4.1
- removed net N$31: R7.2, U1.IN, X3.1
- removed net N$32: R16.2, U1.LEN, U2.Q1
- removed net N$34: JP3.1, U2.D1
- removed net N$8: JP2.2, U1.D1
- removed net N$9: JP2.11, R4.2, U1.FTUNE
- removed net VBB: C13.1, C18.1, C19.1, R10.1, R16.1, R7.1, U1.VBB
- new net +5V: C3.1, C4.1, U$1G$3.VCC
- new net -5V: C1.1, C2.1, U$1G$3.VEE
- new net N$13: R10.2, U$2./CE
- net +3V3: now also R2.1, R7.2, R8.2, U$1G$3.VCC_A, U$1G$3.VCC_B; no longer C1.1, C7.1, C8.1, C9.1, JP4.2, U1.VCC, U1.VCC_2, U1.VCC_3, U1.VCC_4, U2.VCC
- net GND: now also C2.2, C3.2, C4.2, R10.1, R3.2, R4.E, R9.1, U$1G$1.IN-, U$1G$2.IN+, U$1G$2.IN-; no longer C10.2, C13.2, C16.2, C17.2, C18.2, C19.2, C8.2, C9.2, JP1.2, JP2.12, JP4.1, JP4.3, R2.1, R3.1, R4.1, R5.1, R6.2, R8.1, U$1.P$4, U1.VEE, U1.VEE_2, U1.VEE_3, U2.D0, U2.GND, X1.1, X2.1, X2.2, X3.2, X4.2
- net N$1: now also R1.2, U$1G$1.LE; no longer JP2.1, U1.D0
- net N$10: now also R8.1, U$2.TCLD; no longer JP2.3, U1.D2
- net N$11: now also R7.1, U$2./PE; no longer C11.1, R9.1, T1.C
- net N$12: now also R9.2, U$2.MR; no longer C12.1, R8.2, T1.E
- net N$2: now also R2.2, U$1G$1./LE; no longer C3.1, R1.2, U1.Q
- net N$3: now also R3.1, U$1G$1.IN+, X1.1; no longer C2.1, R2.2, U1.~Q
- net N$4: now also R4.A, R4.S, U$1G$1.HYST; no longer C2.2, U$1.P$2
- net N$5: now also R5.1, U$1G$1.Q, U$2.CLK; no longer C3.2, U$1.P$3
- net N$6: now also R6.1, U$1G$1./Q, U$2./CLK; no longer C4.1, U$1.P$1
- net N$7: now also C7.1, R5.2, R6.2, U$2.VBB; no longer C4.2, R3.2, T1.B
Other:
- note removed: "-> Clipping lines, 100ps long"
- note removed: "Copyright 2015 by Mathias Helsen, MIT license"
- moved on the sheet: C1, C2, C3, C4, C5, C6, C7, R1, R10, R2, R3, R5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

Commit message: almost finished prescaled trigger
Parts:
- added C8, C9: (no value), resistor:C-EUC0805
- added X2, X3: BU-SMA-H, con-coax:BU-SMA-H
Connections:
- new net N$14: U$2.COUT, X2.1
- new net N$15: U$2./COUT, X3.1
- net +3V3: now also C8.2, C9.2, U$2.P2, U$2.P3, U$2.P4, U$2.P7, U$2.VCC
- net GND: now also C8.1, C9.1, U$2.P0, U$2.P1, U$2.P5, U$2.P6, U$2.VEE, X2.2, X3.2
Other:
- moved on the sheet: C7, R1, R2, R3, R4, R5, R6, X1

Commit message: almost finished prescaled trigger
Parts:
- added JP1, JP2, JP3: (no value), pinhead:PINHD-1X3
Connections:
- net N$14 renamed TRIGOUT
- net N$15 renamed /TRIGOUT
- net N$3 renamed RFIN
- net N$5 renamed CLKIN
- net N$6 renamed /CLKIN
- net N$7 renamed VBB
- net +3V3: now also JP1.2
- net +5V: now also JP2.2
- net -5V: now also JP3.2
- net GND: now also JP1.1, JP1.3, JP2.1, JP2.3, JP3.1, JP3.3
Changed lines of the file:
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@@
 <part name="GND19" library="supply1" deviceset="GND" device=""/>
 <part name="GND20" library="supply1" deviceset="GND" device=""/>
+<part name="JP1" library="pinhead" deviceset="PINHD-1X3" device=""/>
+<part name="JP2" library="pinhead" deviceset="PINHD-1X3" device=""/>
+<part name="JP3" library="pinhead" deviceset="PINHD-1X3" device=""/>
+<part name="+3V7" library="supply1" deviceset="+3V3" device=""/>
+<part name="P+2" library="supply1" deviceset="+5V" device=""/>
+<part name="P-2" library="supply1" deviceset="-5V" device=""/>
+<part name="GND21" library="supply1" deviceset="GND" device=""/>
 </parts>
 <sheets>
@@
 <instance part="GND19" gate="1" x="165.1" y="88.9"/>
 <instance part="GND20" gate="1" x="165.1" y="111.76"/>
+<instance part="JP1" gate="A" x="205.74" y="50.8"/>
+<instance part="JP2" gate="A" x="205.74" y="35.56"/>
+<instance part="JP3" gate="A" x="205.74" y="20.32"/>
+<instance part="+3V7" gate="G$1" x="190.5" y="50.8" rot="R90"/>
+<instance part="P+2" gate="1" x="190.5" y="35.56" rot="R90"/>
+<instance part="P-2" gate="1" x="190.5" y="20.32" rot="R270"/>
+<instance part="GND21" gate="1" x="198.12" y="7.62"/>
 </instances>
 <busses>
@@
 <pinref part="GND20" gate="1" pin="GND"/>
 </segment>
+<segment>
+<pinref part="JP1" gate="A" pin="1"/>
+<pinref part="GND21" gate="1" pin="GND"/>
+<wire x1="203.2" y1="53.34" x2="198.12" y2="53.34" width="0.1524" layer="91"/>
+<wire x1="198.12" y1="53.34" x2="198.12" y2="48.26" width="0.1524" layer="91"/>
+<pinref part="JP3" gate="A" pin="3"/>
+<wire x1="198.12" y1="48.26" x2="198.12" y2="38.1" width="0.1524" layer="91"/>
+<wire x1="198.12" y1="38.1" x2="198.12" y2="33.02" width="0.1524" layer="91"/>
+<wire x1="198.12" y1="33.02" x2="198.12" y2="22.86" width="0.1524" layer="91"/>
+<wire x1="198.12" y1="22.86" x2="198.12" y2="17.78" width="0.1524" layer="91"/>
+<wire x1="198.12" y1="17.78" x2="198.12" y2="10.16" width="0.1524" layer="91"/>
+<wire x1="203.2" y1="17.78" x2="198.12" y2="17.78" width="0.1524" layer="91"/>
+<junction x="198.12" y="17.78"/>
+<pinref part="JP3" gate="A" pin="1"/>
+<wire x1="203.2" y1="22.86" x2="198.12" y2="22.86" width="0.1524" layer="91"/>
+<junction x="198.12" y="22.86"/>
+<pinref part="JP2" gate="A" pin="3"/>
+<wire x1="203.2" y1="33.02" x2="198.12" y2="33.02" width="0.1524" layer="91"/>
+<junction x="198.12" y="33.02"/>
+<pinref part="JP2" gate="A" pin="1"/>
+<wire x1="203.2" y1="38.1" x2="198.12" y2="38.1" width="0.1524" layer="91"/>
+<junction x="198.12" y="38.1"/>
+<pinref part="JP1" gate="A" pin="3"/>
+<wire x1="203.2" y1="48.26" x2="198.12" y2="48.26" width="0.1524" layer="91"/>
+<junction x="198.12" y="48.26"/>
+</segment>
 </net>
 <net name="+3V3" class="0">
@@
 <pinref part="+3V6" gate="G$1" pin="+3V3"/>
 </segment>
+<segment>
+<pinref part="JP1" gate="A" pin="2"/>
+<pinref part="+3V7" gate="G$1" pin="+3V3"/>
+<wire x1="193.04" y1="50.8" x2="203.2" y2="50.8" width="0.1524" layer="91"/>
+</segment>
 </net>
 <net name="-5V" class="0">
@@
 <junction x="149.86" y="10.16"/>
 </segment>
+<segment>
+<pinref part="JP3" gate="A" pin="2"/>
+<pinref part="P-2" gate="1" pin="-5V"/>
+<wire x1="193.04" y1="20.32" x2="203.2" y2="20.32" width="0.1524" layer="91"/>
+</segment>
 </net>
 <net name="+5V" class="0">
@@
 <junction x="147.32" y="48.26"/>
 </segment>
+<segment>
+<pinref part="JP2" gate="A" pin="2"/>
+<pinref part="P+2" gate="1" pin="+5V"/>
+<wire x1="193.04" y1="35.56" x2="203.2" y2="35.56" width="0.1524" layer="91"/>
+</segment>
 </net>
 <net name="N$1" class="0">
@@
 </segment>
 </net>
-<net name="N$3" class="0">
+<net name="RFIN" class="0">
 <segment>
 <pinref part="U$1" gate="G$1" pin="IN+"/>
@@
 </segment>
 </net>
-<net name="N$5" class="0">
+<net name="CLKIN" class="0">
 <segment>
 <pinref part="U$2" gate="G$1" pin="CLK"/>
@@
 </segment>
 </net>
-<net name="N$6" class="0">
+<net name="/CLKIN" class="0">
 <segment>
 <pinref part="U$2" gate="G$1" pin="/CLK"/>
 <wire x1="109.22" y1="109.22" x2="99.06" y2="109.22" width="0.1524" layer="91"/>
-<wire x1="99.06" y1="109.22" x2="99.06" y2="106.68" width="0.1524" layer="91"/>
+<wire x1="99.06" y1="109.22" x2="96.52" y2="106.68" width="0.1524" layer="91"/>
 <pinref part="R6" gate="G$1" pin="1"/>
-<wire x1="99.06" y1="106.68" x2="86.36" y2="106.68" width="0.1524" layer="91"/>
+<wire x1="96.52" y1="106.68" x2="86.36" y2="106.68" width="0.1524" layer="91"/>
 <wire x1="86.36" y1="106.68" x2="86.36" y2="114.3" width="0.1524" layer="91"/>
 <pinref part="U$1" gate="G$1" pin="/Q"/>
@@
 </segment>
 </net>
-<net name="N$7" class="0">
+<net name="VBB" class="0">
 <segment>
 <pinref part="U$2" gate="G$1" pin="VBB"/>
@@
 </segment>
 </net>
-<net name="N$14" class="0">
+<net name="TRIGOUT" class="0">
 <segment>
 <pinref part="U$2" gate="G$1" pin="COUT"/>
@@
 </segment>
 </net>
-<net name="N$15" class="0">
+<net name="/TRIGOUT" class="0">
 <segment>
 <pinref part="U$2" gate="G$1" pin="/COUT"/>

Commit message: tracking board layout
Parts:
- removed R1: 1k, resistor:R-EU_M0805
- added C10, C11, C12, C13, C14, C15, C16, C17: (no value), resistor:C-EUC0805
- added R11, R12, R18: 1k, resistor:R-EU_M0805
- added R19, R20, R21, R22, R23, R24: (no value), resistor:R-EU_M1206
- added U1, U2, U3: MC100EP32DG, MC100EP32:MC100EP32DG
- R5, R6: device resistor:R-EU_M0805 -> resistor:R-EU_M1206
Connections:
- removed net /TRIGOUT: U$2./COUT, X3.1
- removed net N$1: R1.2, U$1G$1.LE
- removed net N$12: R9.2, U$2.MR
- removed net N$13: R10.2, U$2./CE
- removed net TRIGOUT: U$2.COUT, X2.1
- new net N$15: R18.2, U$1G$1.LE
- new net N$16: C11.1, R21.1, R22.1, U1.VBB
- new net N$17: R21.2, U$1G$1./Q, U1.CLK
- new net N$18: R22.2, U$1G$1.Q, U1.~CLK
- new net N$19: C10.2, R19.1, R20.1, U2.VBB
- new net N$20: R19.2, U1.Q, U2.CLK
- new net N$21: R20.2, U1.~Q, U2.~CLK
- new net N$26: U3.Q, X2.1
- new net N$27: U3.~Q, X3.1
- new net N$28: C12.1, R23.1, R24.1, U3.VBB
- new net N$29: R24.2, U$2./COUT, U3.CLK
- new net N$3: R11.1, U$2.P6
- new net N$30: R23.2, U$2.COUT, U3.~CLK
- new net N$5: R10.1, U$2.P5
- new net N$6: R9.1, U$2.P4
- new net N$7: R12.1, U$2.P7
- net +3V3: now also C13.1, C14.1, C15.1, C16.2, C17.2, R10.2, R11.2, R12.2, R9.2, U1.VCC, U2.VCC, U3.VCC; no longer U$2.P2, U$2.P3, U$2.P4, U$2.P7
- net /CLKIN: now also U2.~Q; no longer U$1G$1./Q
- net CLKIN: now also U2.Q; no longer U$1G$1.Q
- net GND: now also C10.1, C11.2, C12.2, C13.2, C14.2, C15.2, C16.1, C17.1, R18.1, U1.VEE, U2.VEE, U3.VEE; no longer R1.1, R10.1, R9.1, U$2.P0, U$2.P1, U$2.P5, U$2.P6
Other:
- note added: "/ 128"
- note added: "/ 2"
- note added: "/ 4"
- note added: "/ 64"
- moved on the sheet: C7, C8, C9, R10, R2, R3, R4, R5, R6, R7, R8, R9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
